File: HighDRMic_EVB.kicad_sch (KiCad schematic)
At the start: 19 parts, among them J1 Conn_01x02, J10 Conn_01x02, J11 Conn_01x02, J2 Conn_01x02, J3 Conn_01x02, J4 Conn_01x02, J5 Conn_01x02, J6 Conn_01x02, J7 Conn_01x02, J8 Conn_01x02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

Commit message: Added schematic pdf
Other:
- company: (none) -> SKB
- title: (none) -> HighDRMic_EVB
Changed lines of the file:
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@@
 	(generator_version "9.0")
 	(paper "A4")
+	(title_block
+		(title "HighDRMic_EVB")
+		(date "2025-03-06")
+		(rev "v0.1")
+		(company "SKB")
+	)
 	(junction
 		(at 130.81 74.93)
